File: pidp11_cyc1000_adapter.sch (KiCad schematic (older format))
At the start: 2 parts, among them U1 CYC1000

Commit message: all routed
Parts:
- added C1: 0.1uF, Capacitor_SMD:C_0805_2012Metric, symbol Device:C
- added C2: 1uF, Capacitor_SMD:C_0805_2012Metric_Pad1.15x1.40mm_HandSolder, symbol Device:C
- added C3: 0.1uF, Capacitor_SMD:C_0805_2012Metric_Pad1.15x1.40mm_HandSolder, symbol Device:C
- added C4: ??, Capacitor_SMD:C_0805_2012Metric_Pad1.15x1.40mm_HandSolder, symbol Device:C
- added H1, H2, H3, H4: MountingHole, pidp11_cyc1000_adapter:MountingHole_RasPI, symbol Mechanical:MountingHole
- added J2: USB_B_Micro, Connector_USB:USB_Mini-B_Lumberg_2486_01_Horizontal, symbol Connector:USB_B_Micro
- added J3: PMODNIC100, pidp11_cyc1000_adapter:PMOD_2x06, symbol Connector_Generic:Conn_02x06_Top_Bottom
- added J4: Conn_01x02, Connector_PinHeader_2.54mm:PinHeader_1x02_P2.54mm_Horizontal, symbol Connector_Generic:Conn_01x02
- added R1: R, Resistor_SMD:R_0805_2012Metric_Pad1.15x1.40mm_HandSolder, symbol Device:R
- added U2: CP2102, pidp11_cyc1000_adapter:QFN-28-1EP_5x5mm_Pitch0.5mm, symbol pidp11_cyc1000_adapter:CP2102
- added XS1: uSD_ebay, pidp11_cyc1000_adapter:Conn_uSDcard, symbol pidp11_cyc1000_adapter:uSD_ebay
- J1: renamed from J?; footprint (none) -> Connector_PinHeader_2.54mm:PinHeader_2x20_P2.54mm_Vertical
- U1: footprint (none) -> pidp11_cyc1000_adapter:CYC1000
Connections:
- net +3V3: now also U1.26 (3.3V), U1.43 (3.3V), U1.49 (3.3V), C4.1, J3.12 (Pin_12), J3.6 (Pin_6), XS1.4 (Vdd)
- net +5V: now also U1.27 (VIN)
- net GND: now also U1.25 (GND), U1.30 (GND), U1.32 (GND), U1.42 (GND), U1.48 (GND), C1.2, C2.2, C3.2, C4.2, J2.5 (GND), J2.6 (Shield), J3.11 (Pin_11), J3.5 (Pin_5), J4.2 (Pin_2), U2.29 (PAD), U2.3 (GND), XS1.6 (GND)
- net PANEL_COL0: now also U1.45 (PIO_06)
- net PANEL_COL1: now also U1.11 (D2)
- net PANEL_COL10: now also U1.29 (AIN)
- net PANEL_COL11: now also U1.41 (PIO_04)
- net PANEL_COL2: now also U1.14 (D5)
- net PANEL_COL3: now also U1.2 (AIN0)
- net PANEL_COL4: now also U1.47 (PIO_08)
- net PANEL_COL5: now also U1.3 (AIN1)
- net PANEL_COL6: now also U1.4 (AIN2)
- net PANEL_COL7: now also U1.5 (AIN3)
- net PANEL_COL8: now also U1.7 (AIN5)
- net PANEL_COL9: now also U1.31 (AIN7)
- net PANEL_ROW0: now also U1.46 (PIO_07)
- net PANEL_ROW1: now also U1.12 (D3)
- net PANEL_ROW2: now also U1.13 (D4)
- net PANEL_XLED0: now also U1.40 (PIO_03)
- net PANEL_XLED1: now also U1.39 (PIO_02)
- net PANEL_XLED2: now also U1.9 (D0)
- net PANEL_XLED3: now also U1.10 (D1)
- net PANEL_XLED4: now also U1.8 (AIN6)
- net PANEL_XLED5: now also U1.6 (AIN4)
- net ETH_SCLK: now reaches U1.16 (D7)
- net ETH_SCLK: now also J3.4 (Pin_4)
- net ETH_MISO: now reaches U1.17 (D8)
- net ETH_MISO: now also J3.3 (Pin_3)
- net ETH_MOSI: now reaches U1.18 (D9)
- net ETH_MOSI: now also J3.2 (Pin_2)
- net ETH_CS: now reaches U1.19 (D10)
- net ETH_CS: now also J3.1 (Pin_1)
- net SD_MISO: now reaches U1.20 (D11)
- net SD_MISO: now also XS1.7 (DO/DAT0)
- net SD_SCK: now reaches U1.21 (D12)
- net SD_SCK: now also XS1.5 (CLK)
- net SD_MOSI: now reaches U1.22 (D13)
- net SD_MOSI: now also XS1.3 (DI/CMD)
- net SD_CS: now reaches U1.23 (D14)
- net SD_CS: now also XS1.2 (CS/DAT3)
- net RESET: now reaches U1.24 (RESET)
- net RESET: now also J4.1 (Pin_1)
- net UART_RX: now reaches U1.38 (PIO_01)
- net UART_RX: now also U2.26 (TXD)
- net UART_TX: now reaches U1.44 (PIO_05)
- net UART_TX: now also U2.25 (RXD)
- new net: J2.3 (D+), U2.4 (D+)
- new net: J2.2 (D-), U2.5 (D-)
- new net: C2.1, C3.1, J2.1 (VBUS), U2.7 (REGIN), U2.8 (VBUS)
- new net: R1.2, U2.9 (RST)
- new net CP2102_3V3: C1.1, R1.1, U2.6 (VDD)
- new net ETH_INT: J3.7 (Pin_7)
- new net UART_CTS: U2.23 (CTS)
- new net UART_RTS: U2.24 (RTS)
- no-connect marks 11 -> 29
Other:
- note added: "just in case we want some\nbypass cap for the sdcard"
- note added: "not enough pins\nfor CTS/RTS"
- moved on the sheet: J1, U1A, U1B, U1C, U1D, U1E

Commit message: final tweaks before first test run
Parts:
- added J5: HDR_BUTT1, Connector_PinHeader_2.54mm:PinHeader_1x02_P2.54mm_Horizontal, symbol Connector_Generic:Conn_01x02
- added R2: 12K, Resistor_SMD:R_0805_2012Metric_Pad1.15x1.40mm_HandSolder, symbol Device:R
- J4: value Conn_01x02 -> HDR_RESET
Connections:
- net +3V3: now also R2.1
- net ETH_CS: now also U1.18 (D9); no longer U1.19 (D10)
- net ETH_MISO: now also U1.16 (D7); no longer U1.17 (D8)
- net ETH_MOSI: now also U1.17 (D8); no longer U1.18 (D9)
- net ETH_SCLK: now also U1.15 (D6); no longer U1.16 (D7)
- net GND: now also J5.2 (Pin_2)
- new net BUTT1: J5.1 (Pin_1), R2.2, U1.19 (D10)
- no-connect marks 29 -> 34
Other:
- moved on the sheet: C1, C2, C3, C4, J1, J2, J3, J4, R1, U2, XS1
